File: STM32-based Accelerometer Board.kicad_sch (KiCad schematic)
At the start: 12 parts, among them J1 Conn_01x04_Male, U1 ADXL345, U2 STM32F030F4Px, Y1 Crystal

Commit message: Smaller! Think there's low-hanging fruit, but saving status.
Parts:
- U1: JLCPCB Price (none) -> $1.23; JLCPCB Status (none) -> Extended
- U2: JLCPCB Price (none) -> $0.55; JLCPCB Status (none) -> Extended
Connections:
- net ADXL_NCS: now reaches U1.7 (NCS)
- net ADXL_NCS: now also U2.10 (PA4)
Changed lines of the file:
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@@
+    (stroke (width 0) (type default) (color 0 0 0 0))
+  )
+  (wire (pts (xy 93.98 50.038) (xy 96.52 50.038))
     (stroke (width 0) (type default) (color 0 0 0 0))
   )
@@
   )
   (wire (pts (xy 110.49 125.73) (xy 110.49 129.794))
+    (stroke (width 0) (type default) (color 0 0 0 0))
+  )
+  (wire (pts (xy 123.19 145.034) (xy 125.476 145.034))
     (stroke (width 0) (type default) (color 0 0 0 0))
   )
@@
     )
   )
+  (global_label "ADXL_NCS" (shape input) (at 96.52 50.038 0) (fields_autoplaced)
+    (effects (font (size 1.27 1.27)) (justify left))
+    (property "Intersheet References" "${INTERSHEET_REFS}" (id 0) (at 108.3069 49.9586 0)
+      (effects (font (size 1.27 1.27)) (justify left) hide)
+    )
+  )
   (global_label "NRST" (shape input) (at 140.208 40.132 0) (fields_autoplaced)
     (effects (font (size 1.27 1.27)) (justify left))
     (property "Intersheet References" "${INTERSHEET_REFS}" (id 0) (at 147.3987 40.0526 0)
+      (effects (font (size 1.27 1.27)) (justify left) hide)
+    )
+  )
+  (global_label "ADXL_NCS" (shape input) (at 125.476 145.034 0) (fields_autoplaced)
+    (effects (font (size 1.27 1.27)) (justify left))
+    (property "Intersheet References" "${INTERSHEET_REFS}" (id 0) (at 137.2629 144.9546 0)
       (effects (font (size 1.27 1.27)) (justify left) hide)
     )
@@
   )
   (symbol (lib_id "Custom:ADXL345") (at 80.01 25.908 0) (unit 1)
-    (in_bom yes) (on_board yes) (fields_autoplaced)
+    (in_bom yes) (on_board yes)
     (property "Reference" "U1" (id 0) (at 80.01 25.146 0))
     (property "Value" "ADXL345" (id 1) (at 80.01 27.686 0))
@@
       (effects (font (size 1.27 1.27)) hide)
     )
+    (property "JLCPCB Status" "Extended" (id 4) (at 90.17 28.448 0))
+    (property "JLCPCB Price" "$1.23" (id 5) (at 88.392 26.416 0))
     (pin "1")
     (pin "10")
@@
   )
   (symbol (lib_id "MCU_ST_STM32F0:STM32F030F4Px") (at 110.49 147.574 0) (unit 1)
-    (in_bom yes) (on_board yes) (fields_autoplaced)
+    (in_bom yes) (on_board yes)
     (property "Reference" "U2" (id 0) (at 112.5094 168.148 0)
       (effects (font (size 1.27 1.27)) (justify left))
@@
       (effects (font (size 1.27 1.27)) hide)
     )
+    (property "JLCPCB Status" "Extended" (id 4) (at 120.65 130.81 0))
+    (property "JLCPCB Price" "$0.55" (id 5) (at 119.126 128.778 0))
     (pin "1")
     (pin "10")
